File: seggerbreakout.kicad_pcb (KiCad board)
At the start: 2 copper layers, 0 parts

Commit message: Add segger 20pin connector
Parts:
- added P1: SWD, 1pin, F.Cu at (0.00, 0.00)
- added P2: JTAG, SEGGER_INPUT, F.Cu at (199.6, 130.8)
Changed lines of the file:
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@@
 (kicad_pcb (version 3) (host pcbnew "(2013-june-11)-stable")
   (general
-    (links 0)
-    (no_connects 0)
+    (links 1)
+    (no_connects 1)
     (area 0 0 0 0)
     (thickness 1.6)
@@
     (tracks 0)
     (zones 0)
-    (modules 0)
-    (nets 1)
+    (modules 2)
+    (nets 20)
   )
   (page A3)
@@
     (mod_text_width 0.15)
     (pad_size 1.5 1.5)
-    (pad_drill 0.6)
+    (pad_drill 0.6731)
     (pad_to_mask_clearance 0)
     (aux_axis_origin 0 0)
@@
   )
   (net 0 "")
+  (net 1 N-000001)
+  (net 2 N-0000010)
+  (net 3 N-0000011)
+  (net 4 N-0000012)
+  (net 5 N-0000013)
+  (net 6 N-0000014)
+  (net 7 N-0000015)
+  (net 8 N-0000016)
+  (net 9 N-0000017)
+  (net 10 N-0000019)
+  (net 11 N-000002)
+  (net 12 N-0000021)
+  (net 13 N-000003)
+  (net 14 N-000004)
+  (net 15 N-000005)
+  (net 16 N-000006)
+  (net 17 N-000007)
+  (net 18 N-000008)
+  (net 19 N-000009)
   (net_class Default "This is the default net class."
     (clearance 0.254)
@@
     (uvia_drill 0.127)
     (add_net "")
+    (add_net N-000001)
+    (add_net N-0000010)
+    (add_net N-0000011)
+    (add_net N-0000012)
+    (add_net N-0000013)
+    (add_net N-0000014)
+    (add_net N-0000015)
+    (add_net N-0000016)
+    (add_net N-0000017)
+    (add_net N-0000019)
+    (add_net N-000002)
+    (add_net N-0000021)
+    (add_net N-000003)
+    (add_net N-000004)
+    (add_net N-000005)
+    (add_net N-000006)
+    (add_net N-000007)
+    (add_net N-000008)
+    (add_net N-000009)
+  )
+  (module SEGGER_INPUT (layer F.Cu)
+    (at 199.644 130.81)
+    (fp_text reference P2 (at 0 -6.35) (layer F.SilkS)
+      (effects (font (size 1 1) (thickness 0.15)))
+    )
+    (fp_text value JTAG (at 0 5.08) (layer F.SilkS)
+      (effects (font (size 1 1) (thickness 0.15)))
+    )
+    (fp_line (start -2.54 2.54) (end -2.54 3.81) (layer F.SilkS) (width 0.15))
+    (fp_line (start -2.54 3.81) (end -1.27 3.81) (layer F.SilkS) (width 0.15))
+    (fp_line (start -1.27 3.81) (end 2.54 3.81) (layer F.SilkS) (width 0.15))
+    (fp_line (start 2.54 3.81) (end 2.54 2.54) (layer F.SilkS) (width 0.15))
+    (fp_line (start -13.97 2.54) (end -13.97 -5.08) (layer F.SilkS) (width 0.15))
+    (fp_line (start -13.97 -5.08) (end 13.97 -5.08) (layer F.SilkS) (width 0.15))
+    (fp_line (start 13.97 -5.08) (end 13.97 2.54) (layer F.SilkS) (width 0.15))
+    (fp_line (start 13.97 2.54) (end -13.97 2.54) (layer F.SilkS) (width 0.15))
+    (pad 1 thru_hole circle (at -11.43 0) (size 1.5 1.5) (drill 0.6731)
+      (layers *.Cu *.Mask F.SilkS)
+      (net 14 N-000004)
+    )
+    (pad 2 thru_hole circle (at -11.43 -2.54) (size 1.5 1.5) (drill 0.6731)
+      (layers *.Cu *.Mask F.SilkS)
+    )
+    (pad 3 thru_hole circle (at -8.89 0) (size 1.5 1.5) (drill 0.6731)
+      (layers *.Cu *.Mask F.SilkS)
+      (net 15 N-000005)
+    )
+    (pad 4 thru_hole circle (at -8.89 -2.54) (size 1.5 1.5) (drill 0.6731)
+      (layers *.Cu *.Mask F.SilkS)
+      (net 2 N-0000010)
+    )
+    (pad 5 thru_hole circle (at -6.35 0) (size 1.5 1.5) (drill 0.6731)
+      (layers *.Cu *.Mask F.SilkS)
+      (net 1 N-000001)
+    )
+    (pad 6 thru_hole circle (at -6.35 -2.54) (size 1.5 1.5) (drill 0.6731)
+      (layers *.Cu *.Mask F.SilkS)
+      (net 3 N-0000011)
+    )
+    (pad 7 thru_hole circle (at -3.81 0) (size 1.5 1.5) (drill 0.6731)
+      (layers *.Cu *.Mask F.SilkS)
+      (net 16 N-000006)
+    )
+    (pad 8 thru_hole circle (at -3.81 -2.54) (size 1.5 1.5) (drill 0.6731)
+      (layers *.Cu *.Mask F.SilkS)
+      (net 4 N-0000012)
+    )
+    (pad 9 thru_hole circle (at -1.27 0) (size 1.5 1.5) (drill 0.6731)
+      (layers *.Cu *.Mask F.SilkS)
+      (net 17 N-000007)
+    )
+    (pad 10 thru_hole circle (at -1.27 -2.54) (size 1.5 1.5) (drill 0.6731)
+      (layers *.Cu *.Mask F.SilkS)
+      (net 6 N-0000014)
+    )
+    (pad 11 thru_hole circle (at 1.27 0) (size 1.5 1.5) (drill 0.6731)
+      (layers *.Cu *.Mask F.SilkS)
+      (net 19 N-000009)
+    )
+    (pad 12 thru_hole circle (at 1.27 -2.54) (size 1.5 1.5) (drill 0.6731)
+      (layers *.Cu *.Mask F.SilkS)
+      (net 7 N-0000015)
+    )
+    (pad 13 thru_hole circle (at 3.81 0) (size 1.5 1.5) (drill 0.6731)
+      (layers *.Cu *.Mask F.SilkS)
+      (net 18 N-000008)
+    )
+    (pad 14 thru_hole circle (at 3.81 -2.54) (size 1.5 1.5) (drill 0.6731)
+      (layers *.Cu *.Mask F.SilkS)
+      (net 8 N-0000016)
+    )
+    (pad 15 thru_hole circle (at 6.35 0) (size 1.5 1.5) (drill 0.6731)
+      (layers *.Cu *.Mask F.SilkS)
+      (net 5 N-0000013)
+    )
+    (pad 16 thru_hole circle (at 6.35 -2.54) (size 1.5 1.5) (drill 0.6731)
+      (layers *.Cu *.Mask F.SilkS)
+      (net 9 N-0000017)
+    )
+    (pad 17 thru_hole circle (at 8.89 0) (size 1.5 1.5) (drill 0.6731)
+      (layers *.Cu *.Mask F.SilkS)
+      (net 10 N-0000019)
+    )
+    (pad 18 thru_hole circle (at 8.89 -2.54) (size 1.5 1.5) (drill 0.6731)
+      (layers *.Cu *.Mask F.SilkS)
+      (net 11 N-000002)
+    )
+    (pad 19 thru_hole circle (at 11.43 0) (size 1.5 1.5) (drill 0.6731)
+      (layers *.Cu *.Mask F.SilkS)
+      (net 12 N-0000021)
+    )
+    (pad 20 thru_hole circle (at 11.43 -2.54) (size 1.5 1.5) (drill 0.6731)
+      (layers *.Cu *.Mask F.SilkS)
+      (net 13 N-000003)
+    )
+  )
+  (module 1pin (layer F.Cu)
+    (at 0 0)
+    (descr "module 1 pin (ou trou mecanique de percage)")
+    (tags DEV)
+    (fp_text reference P1 (at 0 -3.048) (layer F.SilkS)
+      (effects (font (size 1.016 1.016) (thickness 0.254)))
+    )
+    (fp_text value SWD (at 0 2.794) (layer F.SilkS) hide
+      (effects (font (size 1.016 1.016) (thickness 0.254)))
+    )
+    (fp_circle (center 0 0) (end 0 -2.286) (layer F.SilkS) (width 0.381))
+    (pad 1 thru_hole circle (at 0 0) (size 4.064 4.064) (drill 3.048)
+      (layers *.Cu *.Mask F.SilkS)
+      (net 14 N-000004)
+    )
   )
 )
