File: seggerbreakout.kicad_pcb (KiCad board)
At the start: 2 copper layers, 29.5 x 28 mm, 3 parts, among them P1 SWD, P2 JTAG, P3 JTAG

Commit message: Add final version sent to fab
Parts:
- added G***: OSHW-logo_silkscreen_4mm, OSHW-logo_silkscreen_4mm, F.Cu at (207.3, 120.9)
Routing:
- net /TCK: track 26.6 -> 27.3 mm
Other:
- board text added: "2014-09-12"
- board text removed: "2014-08-31"
